Commit message: homing joint values

File: srdf/panda.srdf.xacro (robot description, xacro)
@@ -14,11 +14,11 @@
     </group>
 <group_state name="home" group="chains">
-        <joint name="panda_joint1" value="0.0"/>
-        <joint name="panda_joint2" value="0.0"/>
-        <joint name="panda_joint3" value="0.0"/>
-        <joint name="panda_joint4" value="0.0"/>
-        <joint name="panda_joint5" value="0.0"/>
-        <joint name="panda_joint6" value="0.0"/>
-        <joint name="panda_joint7" value="0.0"/>
+        <joint name="panda_joint1" value="-0.01782588195099777"/>
+        <joint name="panda_joint2" value="-0.7351092080718704"/>
+        <joint name="panda_joint3" value="0.023999159953865146"/>
+        <joint name="panda_joint4" value="-2.435700656464607"/>
+        <joint name="panda_joint5" value="0.02721460521978436"/>
+        <joint name="panda_joint6" value="1.531987200144168"/>
+        <joint name="panda_joint7" value="0.7534199003476942"/>
 </group_state>
 </robot>
